Commit message: Update HU_L04 leg meshes and foot collision geometry

File: HU_L04_description/urdf/HU_L04_01.urdf (robot description, URDF)
Before this commit: robot HU_L04_01, 39 links, 38 joints
Links:
- link left_ankle_roll_link: mass 1.205462175 -> 1.0092621199999998; geometry collision box size=0.18 0.065 0.022; collision sphere radius=0.005
- link left_hip_yaw_link: mass 2.8471496800000002 -> 2.847143765
- link left_knee_link: mass 5.062820609999999 -> 5.06279911
- link right_ankle_roll_link: mass 1.205462175 -> 1.0092621199999998; geometry collision box size=0.18 0.065 0.022; collision sphere radius=0.005
- link right_hip_yaw_link: mass 2.8471496800000002 -> 2.847143765
- link right_knee_link: mass 5.062820609999999 -> 5.06279911
